File: wave_generator/wave_generator.kicad_sch (KiCad schematic)
At the start: 96 parts, among them J1 KF301_3PIN_POWER, J2 KF301_2PIN_INPUT, J3 KF301_2PIN_INPUT, J4 KF301_2PIN_OUTPUT, J5 UART, J6 SWD, J7 TEST, U1 L7809, U2 LM7909, U3 AMS1117-3.3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

Commit message: PCB not finished yet
Parts:
- J4: footprint Connector_PinHeader_2.54mm:PinHeader_1x04_P2.54mm_Vertical -> myfootprint:KF301-2P
- U8: footprint Package_TO_SOT_SMD:TO-263-2 -> Package_QFP:LQFP-64_10x10mm_P0.5mm
Connections:
- net +3V3: now also C11.1, C12.1, R24.2, TP6.1, U3.2 (VO)
- net +9V: now also TP5.1
- net -9V: now also TP7.1
Other:
- moved on the sheet: C29, C3, C30, C31, C32, C33, C34, C35, C36, C37, C38, C4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
