File: wave_generator/_autosave-wave_generator.kicad_sch (KiCad schematic)
At the start: 100 parts, among them J1 KF301_3PIN_POWER, J2 KF301_2PIN_INPUT, J3 KF301_2PIN_INPUT, J4 KF301_2PIN_OUTPUT, J5 UART, J6 SWD, J7 TEST, U1 L7809, U2 LM7909, U3 AMS1117-3.3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

Commit message: Finished PCB
Parts:
- renumbered D2 to amp1, D3 to freq1, D1 to power1
Changed lines of the file:
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@@
   (symbol (lib_id "Device:LED") (at 216.535 50.165 90) (unit 1)
     (in_bom yes) (on_board yes)
-    (property "Reference" "D1" (id 0) (at 218.821 48.641 90)
+    (property "Reference" "power1" (id 0) (at 218.821 48.641 90)
       (effects (font (size 1.27 1.27)) (justify right))
     )
@@
   (symbol (lib_id "Device:LED") (at 95.25 256.54 90) (unit 1)
     (in_bom yes) (on_board yes)
-    (property "Reference" "D2" (id 0) (at 97.536 255.016 90)
+    (property "Reference" "amp1" (id 0) (at 97.536 255.016 90)
       (effects (font (size 1.27 1.27)) (justify right))
     )
@@
   (symbol (lib_id "Device:LED") (at 113.03 256.54 90) (unit 1)
     (in_bom yes) (on_board yes)
-    (property "Reference" "D3" (id 0) (at 115.316 255.016 90)
+    (property "Reference" "freq1" (id 0) (at 115.316 255.016 90)
       (effects (font (size 1.27 1.27)) (justify right))
     )
@@
       (reference "C38") (unit 1) (value "104") (footprint "Capacitor_SMD:C_0603_1608Metric")
     )
-    (path "/6f149774-e0a5-4122-b56d-41cc05af017d"
-      (reference "D1") (unit 1) (value "LED_RED") (footprint "LED_SMD:LED_0603_1608Metric")
-    )
-    (path "/86d790e1-59c6-42e6-b26b-4004694fc764"
-      (reference "D2") (unit 1) (value "LED_BLUE") (footprint "LED_SMD:LED_0603_1608Metric")
-    )
-    (path "/ce1d41f7-2ab2-4705-abf0-5d3d3e4716b4"
-      (reference "D3") (unit 1) (value "LED_BLUE") (footprint "LED_SMD:LED_0603_1608Metric")
-    )
     (path "/e5926be9-c577-46f6-96cf-d0cd09f7c361"
       (reference "F1") (unit 1) (value "Fuse") (footprint "Fuse:Fuse_1206_3216Metric")
@@
       (reference "X1") (unit 1) (value "16Mhz_Passive_3225") (footprint "Oscillator:Oscillator_SMD_EuroQuartz_XO32-4Pin_3.2x2.5mm")
     )
-  )
+    (path "/86d790e1-59c6-42e6-b26b-4004694fc764"
+      (reference "amp1") (unit 1) (value "LED_BLUE") (footprint "LED_SMD:LED_0603_1608Metric")
+    )
+    (path "/ce1d41f7-2ab2-4705-abf0-5d3d3e4716b4"
+      (reference "freq1") (unit 1) (value "LED_BLUE") (footprint "LED_SMD:LED_0603_1608Metric")
+    )
+    (path "/6f149774-e0a5-4122-b56d-41cc05af017d"
+      (reference "power1") (unit 1) (value "LED_RED") (footprint "LED_SMD:LED_0603_1608Metric")
+    )
+  )
